File: hardware/rmpd_player/rmpd_player.kicad_pcb (KiCad board)
At the start: 2 copper layers, 119.4 x 52.1 mm, 112 parts, among them J1 POWER, J2 PROG, J3 LINE_OUT_INT_1, J4 LINE_OUT, J5 MICRO_SD, J6 POWER_INT, J7 LINE_OUT_INT_2, J8 RESERV, Q1 BC848, Q2 BC848, Q3 BC858, Q4 BC858, U1 DS3231M, U2 VS1011E, U3 LM1117-3.3, U4 ESP32-WROOM, U5 RC4558, U6 RC4558, U7 RC4558, Y1 12.288MHz

Commit message: almost done pcb
Parts:
- added REF**: 1pin, Connectors:1pin, F.Cu at (139.7, 76.2)
- added REF**: 1pin, Connectors:1pin, F.Cu at (139.7, 137.8)
- C10, C11, C13, C14, C16, F1, Q1, Q2, Q3, Q4, R10, R11, R12, R13, R14, R15, R16, R17, R18, R19, R21, R22, R23, R24, R4, R8, R9, U1, U3: moved to B.Cu
- moved Q4 128.5 mm to (80.6, 94.6), turned to 90 degrees
- moved R6 123.3 mm to (84.3, 105.3), turned to 270 degrees
- moved C3 122.8 mm to (61.0, 85.1)
- moved Q2 121.6 mm to (85.7, 85.1), turned to 180 degrees
- moved R11 121.2 mm to (87.5, 99.7), turned to 180 degrees
- moved R3 121.2 mm to (94.2, 109.7)
- moved C13 117.3 mm to (86.4, 89.5), turned to 270 degrees
- moved R12 112.0 mm to (99.8, 99.7)
- moved C17 108.8 mm to (88.9, 92.1)
- moved Q3 107.8 mm to (80.0, 85.1), turned to 180 degrees
- moved C15 107.3 mm to (109.9, 125.1), turned to 270 degrees
- moved R14 106.4 mm to (90.8, 88.3)
- moved R13 105.0 mm to (103.5, 86.9), turned to 270 degrees
- moved Q1 104.1 mm to (90.8, 85.1), turned to 180 degrees
- moved U1 103.7 mm to (60.8, 85.7), turned to 180 degrees
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Connections:
- C4 pad 1: VDDA -> VDD
- C5 pad 1: VDDA -> VDD
- U2 pad 38: VDDA -> VDD
- U2 pad 43: VDDA -> VDD
- U2 pad 45: VDDA -> VDD
Routing:
- net GND: track 216.8 -> 617.1 mm, vias 3 -> 6
- net VDD: track 37.4 -> 284.1 mm, vias 4 -> 15
- net TRANSIENT_MUTE: track 0.00 -> 88.3 mm, vias 0 -> 3
- net I2C_SCL: track 0.00 -> 71.3 mm, vias 0 -> 1
- net I2C_SDA: track 0.00 -> 70.2 mm, vias 0 -> 1
- net OUT_L: track 43.4 -> 112.9 mm, vias 0 -> 3
- net VS_SI: track 0.00 -> 64.0 mm, vias 0 -> 3
- net 5V: track 78.3 -> 137.2 mm, vias 5 -> 7
- net VS_SO: track 0.00 -> 58.3 mm, vias 0 -> 3
- net VS_SCLK: track 0.00 -> 53.0 mm, vias 0 -> 3
- net SD_CLK: track 0.00 -> 52.4 mm, vias 0 -> 3
- net VS_XCS: track 0.00 -> 50.3 mm, vias 0 -> 5
- net SD_D2: track 0.00 -> 44.6 mm, vias 0 -> 2
- net IO0: track 0.00 -> 43.3 mm, vias 0 -> 3
- net EN: track 0.00 -> 42.1 mm, vias 0 -> 4
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Other:
- board outline removed

Commit message: almost done pcb
Parts:
- C3: moved to B.Cu
- moved C3 7.62 mm to (61.0, 92.7)
Routing:
- net GND: track 617.1 -> 637.1 mm, vias 6 -> 15
- net VDD: track 284.1 -> 290.5 mm, vias 15 -> 14
- net Net-(R3-Pad2): track 7.41 -> 8.25 mm
- net Net-(R2-Pad2): track 11.9 -> 12.4 mm
- added copper zone on B.Cu, net GND
- added copper zone on F.Cu, net GND
Other:
- board outline added: 108.6 x 69.2 mm

Commit message: moar pcb
Parts:
- added G***: LOGO_NON_NEG, microsd:LOGO_NON_NEG, F.Cu at (89.5, 78.1)
Routing:
- net GND: track 637.1 -> 698.6 mm
- net VS_XDCS: track 29.4 -> 27.4 mm
- net VS_XRESET: track 40.8 -> 39.0 mm
- net VS_XCS: track 50.3 -> 48.6 mm
- net VS_SCLK: track 53.0 -> 53.6 mm

Commit message: power led
Parts:
- added D2: LED, LEDs:LED_D3.0mm, F.Cu at (85.7, 136.5)
- added R49: 200, Resistors_SMD:R_0805_HandSoldering, B.Cu at (92.7, 137.2)
- moved J6 5.46 mm to (87.4, 130.2)
Routing:
- net VDD: track 290.5 -> 314.8 mm, vias 14 -> 15
- net GND: track 698.6 -> 706.3 mm
- net Net-(D2-Pad2): track 0.00 -> 3.36 mm
- net Net-(F1-Pad1): track 12.8 -> 10.5 mm
Changed lines of the file:
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@@
     (thickness 1.6)
     (drawings 10)
-    (tracks 1066)
+    (tracks 1078)
     (zones 0)
-    (modules 115)
-    (nets 89)
+    (modules 117)
+    (nets 90)
   )
   (page A4)
@@
     (0 F.Cu signal)
     (31 B.Cu signal)
-    (32 B.Adhes user hide)
-    (33 F.Adhes user hide)
-    (34 B.Paste user hide)
-    (35 F.Paste user hide)
+    (32 B.Adhes user)
+    (33 F.Adhes user)
+    (34 B.Paste user)
+    (35 F.Paste user)
     (36 B.SilkS user)
     (37 F.SilkS user)
@@
   (net 87 "Net-(J8-Pad2)")
   (net 88 "Net-(J8-Pad1)")
+  (net 89 "Net-(D2-Pad2)")
   (net_class Default "This is the default net class."
     (clearance 0.2)
@@
     (add_net "Net-(C36-Pad2)")
     (add_net "Net-(C9-Pad1)")
+    (add_net "Net-(D2-Pad2)")
     (add_net "Net-(F1-Pad1)")
     (add_net "Net-(J8-Pad1)")
@@
     (descr "DC Barrel Jack")
     (tags "Power Jack")
-    (fp_text reference J1 (at -8.45 5.75 270) (layer F.SilkS)
+    (fp_text reference J1 (at -11.43 0) (layer F.SilkS)
       (effects (font (size 1 1) (thickness 0.15)))
     )
@@
     (descr "Through hole straight pin header, 1x04, 2.54mm pitch, single row")
     (tags "Through hole pin header THT 1x04 2.54mm single row")
-    (fp_text reference J3 (at 0.635 -2.54) (layer F.SilkS)
+    (fp_text reference J3 (at 2.413 4.191) (layer F.SilkS)
       (effects (font (size 1 1) (thickness 0.15)))
     )
@@
   (module microsd:2RCA (layer F.Cu)
     (at 44.196 141.478)
-    (fp_text reference J4 (at 10.16 -5.461) (layer F.SilkS)
+    (fp_text reference J4 (at 10.414 -2.413) (layer F.SilkS)
       (effects (font (size 1 1) (thickness 0.15)))
     )
@@
   )
   (module Pin_Headers:Pin_Header_Straight_1x02_Pitch2.54mm (layer F.Cu)
-    (at 87.376 135.636 180)
+    (at 87.376 130.175 180)
     (descr "Through hole straight pin header, 1x02, 2.54mm pitch, single row")
     (tags "Through hole pin header THT 1x02 2.54mm single row")
-    (fp_text reference J6 (at 0 -2.33 180) (layer F.SilkS)
+    (fp_text reference J6 (at -0.889 4.445 180) (layer F.SilkS)
       (effects (font (size 1 1) (thickness 0.15)))
     )
@@
       (xy 2.836012 1.27) (xy 2.954325 1.276364)) (layer F.SilkS) (width 0.01))
   )
+  (module Resistors_SMD:R_0805_HandSoldering (layer B.Cu)
+    (at 92.71 137.16 180)
+    (descr "Resistor SMD 0805, hand soldering")
+    (tags "resistor 0805")
+    (attr smd)
+    (fp_text reference R49 (at -3.81 0 180) (layer B.SilkS)
+      (effects (font (size 1 1) (thickness 0.15)) (justify mirror))
+    )
+    (fp_text value 200 (at 0 -1.75 180) (layer B.Fab)
+      (effects (font (size 1 1) (thickness 0.15)) (justify mirror))
+    )
+    (fp_line (start 2.35 -0.9) (end -2.35 -0.9) (layer B.CrtYd) (width 0.05))
+    (fp_line (start 2.35 -0.9) (end 2.35 0.9) (layer B.CrtYd) (width 0.05))
+    (fp_line (start -2.35 0.9) (end -2.35 -0.9) (layer B.CrtYd) (width 0.05))
+    (fp_line (start -2.35 0.9) (end 2.35 0.9) (layer B.CrtYd) (width 0.05))
+    (fp_line (start -0.6 0.88) (end 0.6 0.88) (layer B.SilkS) (width 0.12))
+    (fp_line (start 0.6 -0.88) (end -0.6 -0.88) (layer B.SilkS) (width 0.12))
+    (fp_line (start -1 0.62) (end 1 0.62) (layer B.Fab) (width 0.1))
+    (fp_line (start 1 0.62) (end 1 -0.62) (layer B.Fab) (width 0.1))
+    (fp_line (start 1 -0.62) (end -1 -0.62) (layer B.Fab) (width 0.1))
+    (fp_line (start -1 -0.62) (end -1 0.62) (layer B.Fab) (width 0.1))
+    (fp_text user %R (at 0 0 180) (layer B.Fab)
+      (effects (font (size 0.5 0.5) (thickness 0.075)) (justify mirror))
+    )
+    (pad 2 smd rect (at 1.35 0 180) (size 1.5 1.3) (layers B.Cu B.Paste B.Mask)
+      (net 89 "Net-(D2-Pad2)"))
+    (pad 1 smd rect (at -1.35 0 180) (size 1.5 1.3) (layers B.Cu B.Paste B.Mask)
+      (net 5 VDD))
+    (model ${KISYS3DMOD}/Resistors_SMD.3dshapes/R_0805.wrl
+      (at (xyz 0 0 0))
+      (scale (xyz 1 1 1))
+      (rotate (xyz 0 0 0))
+    )
+  )
+  (module LEDs:LED_D3.0mm (layer F.Cu)
+    (at 85.725 136.525)
+    (descr "LED, diameter 3.0mm, 2 pins")
+    (tags "LED diameter 3.0mm 2 pins")
+    (fp_text reference D2 (at 1.27 -2.96) (layer F.SilkS)
+      (effects (font (size 1 1) (thickness 0.15)))
+    )
+    (fp_text value LED (at 1.27 2.96) (layer F.Fab)
+      (effects (font (size 1 1) (thickness 0.15)))
+    )
+    (fp_line (start 3.7 -2.25) (end -1.15 -2.25) (layer F.CrtYd) (width 0.05))
+    (fp_line (start 3.7 2.25) (end 3.7 -2.25) (layer F.CrtYd) (width 0.05))
+    (fp_line (start -1.15 2.25) (end 3.7 2.25) (layer F.CrtYd) (width 0.05))
+    (fp_line (start -1.15 -2.25) (end -1.15 2.25) (layer F.CrtYd) (width 0.05))
+    (fp_line (start -0.29 1.08) (end -0.29 1.236) (layer F.SilkS) (width 0.12))
+    (fp_line (start -0.29 -1.236) (end -0.29 -1.08) (layer F.SilkS) (width 0.12))
+    (fp_line (start -0.23 -1.16619) (end -0.23 1.16619) (layer F.Fab) (width 0.1))
+    (fp_circle (center 1.27 0) (end 2.77 0) (layer F.Fab) (width 0.1))
+    (fp_arc (start 1.27 0) (end 0.229039 1.08) (angle -87.9) (layer F.SilkS) (width 0.12))
+    (fp_arc (start 1.27 0) (end 0.229039 -1.08) (angle 87.9) (layer F.SilkS) (width 0.12))
+    (fp_arc (start 1.27 0) (end -0.29 1.235516) (angle -108.8) (layer F.SilkS) (width 0.12))
+    (fp_arc (start 1.27 0) (end -0.29 -1.235516) (angle 108.8) (layer F.SilkS) (width 0.12))
+    (fp_arc (start 1.27 0) (end -0.23 -1.16619) (angle 284.3) (layer F.Fab) (width 0.1))
+    (pad 2 thru_hole circle (at 2.54 0) (size 1.8 1.8) (drill 0.9) (layers *.Cu *.Mask)
+      (net 89 "Net-(D2-Pad2)"))
+    (pad 1 thru_hole rect (at 0 0) (size 1.8 1.8) (drill 0.9) (layers *.Cu *.Mask)
+      (net 2 GND))
+    (model ${KISYS3DMOD}/LEDs.3dshapes/LED_D3.0mm.wrl
+      (at (xyz 0 0 0))
+      (scale (xyz 0.393701 0.393701 0.393701))
+      (rotate (xyz 0 0 0))
+    )
+  )
   (dimension 69.215 (width 0.3) (layer Dwgs.User)
     (gr_text "69.215 mm" (at 154.5 106.9975 270) (layer Dwgs.User)
@@
   (segment (start 86.775 86.04) (end 88.450001 84.364999) (width 0.25) (layer B.Cu) (net 2) (status 10))
   (segment (start 86.725 86.04) (end 86.775 86.04) (width 0.25) (layer B.Cu) (net 2) (status 30))
-  (segment (start 93.98 135.635) (end 93.98 133.635) (width 0.25) (layer B.Cu) (net 2) (status 20))
-  (segment (start 93.979 135.636) (end 93.98 135.635) (width 0.25) (layer B.Cu) (net 2))
-  (segment (start 87.376 135.636) (end 93.979 135.636) (width 0.25) (layer B.Cu) (net 2) (status 10))
   (segment (start 86.1 101.6) (end 86.2 101.6) (width 0.25) (layer F.Cu) (net 2) (status 30))
   (segment (start 84.328 103.372) (end 86.1 101.6) (width 0.25) (layer F.Cu) (net 2) (status 30))
@@
   (segment (start 139.7 86.725) (end 136.255 90.17) (width 0.25) (layer F.Cu) (net 2))
   (segment (start 139.7 76.2) (end 139.7 86.725) (width 0.25) (layer F.Cu) (net 2))
+  (segment (start 91.98 133.635) (end 93.98 133.635) (width 0.25) (layer B.Cu) (net 2))
+  (segment (start 89.736 133.635) (end 91.98 133.635) (width 0.25) (layer B.Cu) (net 2))
+  (segment (start 87.376 131.275) (end 89.736 133.635) (width 0.25) (layer B.Cu) (net 2))
+  (segment (start 87.376 130.175) (end 87.376 131.275) (width 0.25) (layer B.Cu) (net 2))
+  (segment (start 86.276 130.175) (end 87.376 130.175) (width 0.25) (layer B.Cu) (net 2))
+  (segment (start 85.725 130.726) (end 86.276 130.175) (width 0.25) (layer B.Cu) (net 2))
+  (segment (start 85.725 136.525) (end 85.725 130.726) (width 0.25) (layer B.Cu) (net 2))
   (segment (start 94.095 112.3) (end 94.095 114.013002) (width 0.25) (layer B.Cu) (net 3) (status 10))
   (segment (start 95.33 115.248002) (end 95.33 116.205) (width 0.25) (layer B.Cu) (net 3) (status 20))
@@
   (segment (start 129.609315 88.9) (end 125.73 92.779315) (width 0.25) (layer B.Cu) (net 5))
   (segment (start 130.175 88.9) (end 129.609315 88.9) (width 0.25) (layer B.Cu) (net 5))
+  (via (at 99.695 138.43) (size 0.8) (drill 0.4) (layers F.Cu B.Cu) (net 5))
+  (segment (start 94.06 137.16) (end 98.425 137.16) (width 0.25) (layer B.Cu) (net 5))
+  (segment (start 98.425 137.16) (end 99.695 138.43) (width 0.25) (layer B.Cu) (net 5))
+  (segment (start 108.805 125.095) (end 109.855 125.095) (width 0.25) (layer F.Cu) (net 5))
+  (segment (start 108.729999 125.170001) (end 108.805 125.095) (width 0.25) (layer F.Cu) (net 5))
+  (segment (start 108.729999 129.395001) (end 108.729999 125.170001) (width 0.25) (layer F.Cu) (net 5))
+  (segment (start 99.695 138.43) (end 108.729999 129.395001) (width 0.25) (layer F.Cu) (net 5))
   (segment (start 132.88 90.17) (end 132.755 90.17) (width 0.25) (layer F.Cu) (net 6) (status 30))
   (segment (start 134.785 88.265) (end 132.88 90.17) (width 0.25) (layer F.Cu) (net 6) (status 30))
@@
   (segment (start 93.795 127.45) (end 93.98 127.635) (width 0.25) (layer B.Cu) (net 13) (status 30))
   (segment (start 93.795 123.825) (end 93.795 127.45) (width 0.25) (layer B.Cu) (net 13) (status 30))
-  (segment (start 92.837 127.635) (end 93.98 127.635) (width 0.25) (layer B.Cu) (net 13) (status 30))
-  (segment (start 87.376 133.096) (end 92.837 127.635) (width 0.25) (layer B.Cu) (net 13) (status 30))
+  (segment (start 87.376 127.635) (end 93.98 127.635) (width 0.25) (layer B.Cu) (net 13))
   (via (at 128.27 121.83) (size 0.8) (drill 0.4) (layers F.Cu B.Cu) (net 14))
   (via (at 133.470748 123.877066) (size 0.8) (drill 0.4) (layers F.Cu B.Cu) (net 14))
@@
   (segment (start 119.677 83.482) (end 119.38 83.185) (width 0.25) (layer F.Cu) (net 88) (status 30))
   (segment (start 119.677 93.616) (end 119.677 83.482) (width 0.25) (layer F.Cu) (net 88) (status 30))
+  (segment (start 90.725 136.525) (end 91.36 137.16) (width 0.25) (layer B.Cu) (net 89))
+  (segment (start 88.265 136.525) (end 90.725 136.525) (width 0.25) (layer B.Cu) (net 89))
   (zone (net 2) (net_name GND) (layer B.Cu) (hatch edge 0.508)
     (connect_pads (clearance 0.508))
